File: PSF-A85_Souliss_Prototype/eagle/esp8285/mainTest.brd (EAGLE design)
At the start: 100 x 80 mm, 53 parts, among them IC2 PCF8574P, IC3 PCF8591P, IC4 75176AP, Q1 2N7000, U1 PSF-A85, U2 V_REG_MC33269DT, X1 22-23-2031, X2 RS485_TERMINATOR, X3 I test point.

Commit message: Optimice work pending
SCHEMATIC AND PCB
Parts:
- moved SV5 75.4 mm to (85.1, 12.7), turned to 0 degrees
- moved U$1 56.6 mm to (1.27, 55.9)
Routing:
- net PIN_HEADER8: track 10.5 -> 0.00 mm
- net PIN_HEADER7: track 6.34 -> 0.00 mm
- net PIN_HEADER6: track 5.22 -> 0.00 mm
- net PIN_HEADER5: track 1.63 -> 0.00 mm
Changed lines of the file:
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@@
 </element>
 <element name="U2" library="SparkFun-PowerIC" package="DPAK" value="V_REG_MC33269DT" x="67.31" y="72.39"/>
-<element name="SV5" library="con-lsta" package="FE09" value="" x="24.13" y="57.15" rot="R90">
-<attribute name="MF" value="" x="24.13" y="57.15" size="1.778" layer="27" rot="R90" display="off"/>
-<attribute name="OC_FARNELL" value="unknown" x="24.13" y="57.15" size="1.778" layer="27" rot="R90" display="off"/>
-<attribute name="OC_NEWARK" value="unknown" x="24.13" y="57.15" size="1.778" layer="27" rot="R90" display="off"/>
-<attribute name="MPN" value="" x="24.13" y="57.15" size="1.778" layer="27" rot="R90" display="off"/>
+<element name="SV5" library="con-lsta" package="FE09" value="" x="85.09" y="12.7">
+<attribute name="MF" value="" x="85.09" y="12.7" size="1.778" layer="27" display="off"/>
+<attribute name="OC_FARNELL" value="unknown" x="85.09" y="12.7" size="1.778" layer="27" display="off"/>
+<attribute name="OC_NEWARK" value="unknown" x="85.09" y="12.7" size="1.778" layer="27" display="off"/>
+<attribute name="MPN" value="" x="85.09" y="12.7" size="1.778" layer="27" display="off"/>
 </element>
-<element name="U$1" library="ITEAD" package="PCB-2G4-ANTENNA" value="PCB-2G4-ANTENNA" x="-7.62" y="0"/>
+<element name="U$1" library="ITEAD" package="PCB-2G4-ANTENNA" value="PCB-2G4-ANTENNA" x="1.27" y="55.88"/>
 </elements>
 <signals>
@@
 <contactref element="U1" pad="P$5"/>
 <contactref element="SV5" pad="1"/>
-<wire x1="24.13" y1="46.99" x2="15.24" y2="53.34" width="0" layer="19" extent="1-1"/>
+<wire x1="74.93" y1="12.7" x2="15.24" y2="53.34" width="0" layer="19" extent="1-1"/>
 </signal>
 <signal name="PIN_HEADER1">
 <contactref element="U1" pad="P$6"/>
 <contactref element="SV5" pad="2"/>
-<wire x1="24.13" y1="49.53" x2="16.51" y2="53.34" width="0" layer="19" extent="1-1"/>
+<wire x1="77.47" y1="12.7" x2="16.51" y2="53.34" width="0" layer="19" extent="1-1"/>
 </signal>
 <signal name="PIN_HEADER2">
 <contactref element="U1" pad="P$7"/>
 <contactref element="SV5" pad="3"/>
-<wire x1="24.13" y1="52.07" x2="17.78" y2="53.34" width="0" layer="19" extent="1-1"/>
+<wire x1="80.01" y1="12.7" x2="17.78" y2="53.34" width="0" layer="19" extent="1-1"/>
 </signal>
 <signal name="PIN_HEADER3">
 <contactref element="U1" pad="P$13"/>
 <contactref element="SV5" pad="4"/>
-<wire x1="24.13" y1="54.61" x2="20.066" y2="60.706" width="0" layer="19" extent="1-1"/>
+<wire x1="82.55" y1="12.7" x2="20.066" y2="60.706" width="0" layer="19" extent="1-1"/>
 </signal>
 <signal name="PIN_HEADER4">
 <contactref element="U1" pad="P$14"/>
 <contactref element="SV5" pad="5"/>
-<wire x1="24.13" y1="57.15" x2="20.066" y2="61.976" width="0" layer="19" extent="1-1"/>
+<wire x1="85.09" y1="12.7" x2="20.066" y2="61.976" width="0" layer="19" extent="1-1"/>
 </signal>
 <signal name="PIN_HEADER5">
 <contactref element="U1" pad="P$15"/>
 <contactref element="SV5" pad="6"/>
-<wire x1="20.066" y1="63.246" x2="20.32" y2="63.5" width="0.4064" layer="1"/>
-<wire x1="20.32" y1="63.5" x2="21.59" y2="63.5" width="0.4064" layer="1"/>
-<wire x1="21.59" y1="63.5" x2="24.13" y2="59.69" width="0" layer="19" extent="1-16"/>
+<wire x1="20.066" y1="63.246" x2="87.63" y2="12.7" width="0" layer="19" extent="1-1"/>
 </signal>
 <signal name="PIN_HEADER6">
 <contactref element="U1" pad="P$16"/>
 <contactref element="SV5" pad="7"/>
-<wire x1="20.066" y1="64.516" x2="20.32" y2="64.77" width="0.4064" layer="1"/>
-<wire x1="20.32" y1="64.77" x2="21.59" y2="64.77" width="0.4064" layer="1"/>
-<wire x1="21.59" y1="64.77" x2="24.13" y2="62.23" width="0.4064" layer="1"/>
+<wire x1="20.066" y1="64.516" x2="90.17" y2="12.7" width="0" layer="19" extent="1-1"/>
 </signal>
 <signal name="PIN_HEADER8">
 <contactref element="U1" pad="P$18"/>
 <contactref element="SV5" pad="9"/>
-<wire x1="24.13" y1="67.31" x2="24.13" y2="68.58" width="0.4064" layer="1"/>
-<wire x1="24.13" y1="68.58" x2="22.86" y2="69.85" width="0.4064" layer="1"/>
-<wire x1="22.86" y1="69.85" x2="19.05" y2="69.85" width="0.4064" layer="1"/>
-<wire x1="19.05" y1="69.85" x2="17.78" y2="68.58" width="0.4064" layer="1"/>
-<wire x1="17.78" y1="68.58" x2="17.78" y2="66.802" width="0.4064" layer="1"/>
+<wire x1="17.78" y1="66.802" x2="95.25" y2="12.7" width="0" layer="19" extent="1-1"/>
 </signal>
 <signal name="PIN_HEADER7">
 <contactref element="U1" pad="P$17"/>
 <contactref element="SV5" pad="8"/>
-<wire x1="19.05" y1="66.802" x2="19.558" y2="67.31" width="0.4064" layer="1"/>
-<wire x1="19.558" y1="67.31" x2="20.32" y2="67.31" width="0.4064" layer="1"/>
-<wire x1="20.32" y1="67.31" x2="22.86" y2="64.77" width="0.4064" layer="1"/>
-<wire x1="22.86" y1="64.77" x2="24.13" y2="64.77" width="0.4064" layer="1"/>
+<wire x1="19.05" y1="66.802" x2="92.71" y2="12.7" width="0" layer="19" extent="1-1"/>
 </signal>
 <signal name="N$32">
@@
 <contactref element="U$1" pad="1"/>
 <contactref element="U1" pad="P$1"/>
-<wire x1="-7.32" y1="0" x2="10.16" y2="53.34" width="0" layer="19" extent="1-1"/>
+<wire x1="1.57" y1="55.88" x2="10.16" y2="53.34" width="0" layer="19" extent="1-1"/>
 </signal>
 </signals>
